File: PCB/Model K Pico-0.2.kicad_sch (KiCad schematic)
At the start: 175 parts, among them SW1 SW_SPST

Commit message: kmk and pcb updates
Connections:
- net SCL: now also RPI1.2 (GPIO1); no longer RPI1.1 (GPIO0)
- net SDA: now also RPI1.1 (GPIO0); no longer RPI1.2 (GPIO1)
Changed lines of the file:
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@@
     (effects (font (size 1.27 1.27)) (justify right bottom))
   )
-  (label "SDA" (at 201.93 198.12 180)
+  (label "SDA" (at 201.93 195.58 180)
     (effects (font (size 1.27 1.27)) (justify right bottom))
   )
@@
     (effects (font (size 1.27 1.27)) (justify right bottom))
   )
-  (label "SCL" (at 201.93 195.58 180)
+  (label "SCL" (at 201.93 198.12 180)
     (effects (font (size 1.27 1.27)) (justify right bottom))
   )
